Commit message: Add joint position controller

File: rbvogui_description/robots/rbvogui_realsense_ur5.urdf.xacro (robot description, xacro)
@@ -94,5 +94,5 @@
         <xacro:include filename="$(find rbvogui_description)/realsense/d435.urdf.xacro" />
         <sensor_d435 parent="${prefix}arm_wrist_3_link">
-            <origin xyz="0 0 0" rpy="0 0 0"/>
+            <origin xyz="0 0 0" rpy="0 -1.57 0"/>
         </sensor_d435>
     </xacro:macro>
